File: hw/bowlThrusterControl/bowlThrusterControl.sch (KiCad schematic (older format))
At the start: 22 parts, among them IC1 L298, P1 INPUT_1, P2 INPUT_2, P3 Battery, P4 OUTPUT_1, P5 OUTPUT_2, T1 BC547, T2 BC547

Commit message: Fix PCB
Connections:
- wire segments 49 -> 52
Other:
- moved on the sheet: R1, R2

Commit message: Made a note for tudor
Other:
- note added: "VCC and VSS is swapped"
Changed lines of the file:
@@
-EESchema Schematic File Version 2  date man 12 nov 2012 15:05:27 CET
+EESchema Schematic File Version 2  date man 12 nov 2012 20:13:02 CET
 LIBS:power
 LIBS:device
@@
 Comment4 ""
 $EndDescr
+Text Notes 5050 1300 0    60   ~ 0
+VCC and VSS is swapped
 Wire Wire Line
 	3500 3400 3500 3050

Commit message: Redo of mistaken board
Other:
- note removed: "VCC and VSS is swapped"
- moved on the sheet: C1
