File: hw/icp/icp.kicad_pcb (KiCad board)
At the start: 2 copper layers, 5 parts

Commit message: More ICP
Parts:
- removed BANANA_PANEL (x2): Val*, BANANA_PANEL
- removed JST-XH_TOP_ENTRY (x2): Val*, JST-XH_TOP_ENTRY
- added BZ1: KX1205, KX1205, F.Cu at (40.6, 158.8)
- added C1: 100n, SM0805, F.Cu at (64.8, 179.1)
- added C10: 100n, SM0805, F.Cu at (114.3, 171.4)
- added C11: 22p, SM0805, F.Cu at (123.2, 64.8)
- added C12: 22p, SM0805, F.Cu at (116.8, 64.8)
- added C2: 100n, SM0805, F.Cu at (99.1, 171.4)
- added C3: 100n, SM0805, F.Cu at (74.9, 179.1)
- added C4: 100n, SM0805, F.Cu at (40.6, 179.1)
- added C5: 100n, SM0805, F.Cu at (85.1, 179.1)
- added C6: 100n, SM0805, F.Cu at (45.7, 179.1)
- added C7: 100n, SM0805, F.Cu at (95.2, 179.1)
- added C8: 100n, SM0805, F.Cu at (55.9, 179.1)
- added C9: 100n, SM0805, F.Cu at (80.0, 179.1)
- added D1: Alarm, LED-1206-header, F.Cu at (141.0, 33.0)
- added D2: ON, LED-1206-header, F.Cu at (120.7, 33.0)
- added D3: Sample, LED-1206-header, F.Cu at (127.0, 33.0)
- added D4: Data, LED-1206-header, F.Cu at (134.6, 33.0)
- added D5: AUX, LED-1206-header, F.Cu at (147.3, 33.0)
- added IC1: ATMEGA168P-20AU, TQFP32, B.Cu at (133.3, 72.4)
- added K1: Tacho0, SIL-3, F.Cu at (87.6, 167.6)
- added K2: Tacho1, SIL-3, F.Cu at (78.7, 167.6)
- added L1: 10µ, SM0805, F.Cu at (128.3, 176.5)
- added P1: PX0707/06S, PX0707/P/6, B.Cu at (190.0, 72.5)
- added P10: UART, SIL-6, F.Cu at (133.3, 96.5)
- added P11: WLD2, SIL-2, F.Cu at (153.7, 43.2)
- added P2: PX0707/06S, PX0707/P/6, B.Cu at (80.0, 72.5)
- added P3: Deans Male, bornier2, F.Cu at (250.2, 45.7)
- added P4: Deans Male, bornier2, F.Cu at (43.2, 45.7)
- added P5: JST-XH, JST-XH_TOP_ENTRY, F.Cu at (250.2, 64.8)
- added P6: JST-XH, JST-XH_TOP_ENTRY, F.Cu at (44.5, 73.7)
- added P7: WLD1, SIL-2, F.Cu at (135.9, 49.5)
- added P8: I²C, SIL-4, F.Cu at (110.5, 80.0)
- added P9: 5V PWR, SIL-4, F.Cu at (113.0, 94.0)
- added Q1: BC846, SOT23EBC, B.Cu at (149.9, 47.0)
- added Q2: BC846, SOT23EBC, B.Cu at (142.2, 48.3)
- added Q3: BC846, SOT23EBC, B.Cu at (147.3, 53.3)
- added Q4: BC846, SOT23EBC, B.Cu at (141.0, 54.6)
- added R1: 7K5, SM0805, F.Cu at (114.3, 176.5)
- added R10: 1K3, SM0805, F.Cu at (109.2, 171.4)
- added R11: 9K1, SM0805, F.Cu at (90.2, 176.5)
- added R12: 330R, SM0805, F.Cu at (85.1, 176.5)
- added R13: 910R, SM0805, F.Cu at (80.0, 176.5)
- added R14: 9K1, SM0805, F.Cu at (104.1, 176.5)
- added R15: 330R, SM0805, F.Cu at (40.6, 176.5)
- added R16: 910R, SM0805, F.Cu at (35.6, 176.5)
- added R17: 9K1, SM0805, F.Cu at (74.9, 176.5)
- added R18: 560R, SM0805, F.Cu at (69.8, 176.5)
- added R19: 680R, SM0805, F.Cu at (64.8, 176.5)
- added R2: 2K7, SM0805, F.Cu at (109.2, 176.5)
- added R20: 9K1, SM0805, F.Cu at (128.3, 171.4)
- added R21: 560R, SM0805, B.Cu at (61.0, 171.4)
- added R22: 680R, SM0805, F.Cu at (119.4, 171.4)
- added R23: 100R, SM0805, F.Cu at (69.8, 179.1)
- added R24: 100R, SM0805, F.Cu at (124.5, 171.4)
- added R25: 100R, SM0805, F.Cu at (35.6, 179.1)
- added R26: 100R, SM0805, F.Cu at (109.2, 179.1)
- added R27: 100R, SM0805, F.Cu at (90.2, 179.1)
- added R28: 100R, SM0805, F.Cu at (50.8, 179.1)
- added R29: 100R, SM0805, F.Cu at (99.1, 179.1)
- added R30: 100R, SM0805, F.Cu at (61.0, 179.1)
- added R31: R, SM0805, F.Cu at (124.5, 176.5)
- added R32: R, SM0805, F.Cu at (85.1, 171.4)
- added R33: 4K7, SM0805, F.Cu at (95.2, 176.5)
- added R34: R, SM0805, F.Cu at (80.0, 171.4)
- added R35: 4K7, SM0805, F.Cu at (114.3, 179.1)
- added R36: R, SM0805, F.Cu at (119.4, 176.5)
- added R37: R, SM0805, F.Cu at (55.9, 176.5)
- added R38: 4K7, SM0805, B.Cu at (146.1, 45.7)
- added R39: 4K7, SM0805, B.Cu at (152.4, 52.1)
- added R4: 2K7, SM0805, B.Cu at (69.8, 171.4)
- added R5: 9K1, SM0805, F.Cu at (45.7, 176.5)
- added R6: 91R, SM0805, F.Cu at (99.1, 176.5)
- added R7: 1K3, SM0805, F.Cu at (50.8, 176.5)
- added R8: 9K1, SM0805, B.Cu at (66.0, 171.4)
- added R9: 91R, SM0805, F.Cu at (104.1, 171.4)
- added X1: 16MHz, HC-49V, F.Cu at (119.4, 68.6)
- R3: value Val* -> 7K5; footprint R3 -> SM0805; moved to B.Cu
- moved R3 138.9 mm to (74.9, 171.4)
Connections:
- R3 pad 1: (no net) -> N-0000055
- R3 pad 2: (no net) -> N-0000012
Other:
- board outline added: 240 x 90 mm

Commit message: Add comment
Parts:
- C11, C12: moved to B.Cu
- moved R25 192.5 mm to (208.3, 94.0), turned to 270 degrees
- moved C1 185.7 mm to (221.0, 78.7), turned to 270 degrees
- moved R5 181.8 mm to (205.7, 90.2), turned to 270 degrees
- moved R7 181.8 mm to (210.8, 90.2), turned to 270 degrees
- moved R23 179.3 mm to (218.4, 78.7), turned to 90 degrees
- moved C3 160.3 mm to (210.8, 94.0), turned to 90 degrees
- moved R37 153.3 mm to (135.9, 45.7), turned to 270 degrees
- moved R2 144.7 mm to (215.9, 78.7), turned to 90 degrees
- moved R32 143.2 mm to (153.7, 45.7), turned to 270 degrees
- moved R19 142.9 mm to (161.3, 71.1), turned to 270 degrees
- moved R34 141.4 mm to (144.8, 45.7), turned to 270 degrees
- moved R18 141.2 mm to (163.8, 71.1), turned to 90 degrees
- moved R17 139.5 mm to (166.4, 71.1), turned to 270 degrees
- moved BZ1 139.3 mm to (135.9, 57.1), turned to 270 degrees
- moved R6 139.2 mm to (208.3, 90.2), turned to 90 degrees
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Connections:
- R13 pad 2: (no net) -> GND
- R19 pad 2: (no net) -> GND
- R2 pad 2: (no net) -> GND
- R7 pad 2: (no net) -> GND
Routing:
- net N-0000051: track 0.00 -> 20.3 mm
- net N-0000052: track 0.00 -> 19.3 mm
- net N-0000062: track 0.00 -> 7.96 mm
- net N-0000061: track 0.00 -> 7.83 mm
